File: BirdBox1/BirdBox1.kicad_sch (KiCad schematic)
At the start: 12 parts, among them J1 Raspberry Pi 2x20 Conn, J2 1x2 female, J2b 1x2 male, J4 1x6 female, J4 1x6 male

Commit message: Recent changes to 2025 versions
Parts:
- added J3: 01x04 Male, symbol Connector:Conn_01x04_Male
Connections:
- net GND: no longer J1.11 (GPIO17), J4.6 (Pin_6)
- net at J1.15 (GPIO22): now also J3.4 (Pin_4)
- net at J1.26 (~{CE1}/GPIO7): now also J3.3 (Pin_3)
- net at J1.29 (GCLK1/GPIO5): no longer R2.1
- net at J1.32 (PWM0/GPIO12): now also J3.2 (Pin_2)
- net at J1.33 (PWM1/GPIO13): now also J3.1 (Pin_1)
- net at J1.7 (GCLK0/GPIO4): now also R2.1
- new net: J1.11 (GPIO17), J4.6 (Pin_6)
- new net: J4.2 (Pin_2), MIC1.2 (GND)
- new net: J4.3 (Pin_3), MIC1.3 (BCLK)
- new net: J4.4 (Pin_4), MIC1.4 (DOUT)
- new net: J4.5 (Pin_5), MIC1.5 (LRCLK)
- new net: J4.6 (Pin_6), MIC1.6 (SEL)
Other:
- note added: "GPIOs for Clipper 4G LTE Mini Hat: 5 - SW_A 6 - 3V3_PWRKEY 14 - 3V3_UART_LTES_RX 15 - 3V3_UART_LTES_TX 16 - SW_B 24 - 3V3_RESET 25 - 3V3_NETLIGHT"
