File: STM32U031_board/STM32U031_board.kicad_sch (KiCad schematic)
At the start: 0 parts

Commit message: Snapshot:
- after adding L1 inductor package
Other:
- sheet Connectors, LEDs, pushbutton ports: added PA10/RX, PA13/SWDIO, PA14/SWCLK, PA9/TX, PB6/SCL, PB7/SDA, PF3; removed none
- sheet Headers ports: added EN, PA0, PA1, PA10, PA11, PA12, PA13, PA14, PA15, PA2, PA3, PA4, PA5, PA6, PA7, PA8, PA9, PB0, PB1, PB3, PB4, PB5, PB6, PB7, PC14, PC15, PF2, PF3; removed none
- sheet MCU ports: added PA0, PA1, PA10/RX, PA11, PA12, PA13/SWDIO, PA14/SWCLK, PA15, PA2, PA3, PA4, PA5, PA6, PA7, PA8, PA9/TX, PB0, PB1, PB3, PB4, PB5, PB6/SCL, PB7/SDA, PC14, PC15, PF2, PF3; removed none
- sheet Power supply ports: added EN, PGOOD; removed none
