File: STM32U031_board/misc.kicad_sch (KiCad schematic)
At the start: 6 parts, among them J3 SWD, J4 UART, J6 QT/ST, SW1 User pushbutton

Commit message: Snapshot:
- after adding L1 inductor package
Parts:
- J5: renamed from J6; footprint Connector_JST:JST_SH_BM04B-SRSS-TB_1x04-1MP_P1.00mm_Vertical -> Connector_JST:JST_SH_SM04B-SRSS-TB_1x04-1MP_P1.00mm_Horizontal
