File: STM32U031_board/MCU.kicad_sch (KiCad schematic)
At the start: 1 part, among them U1 STM32U031K8Ux

Commit message: Checkin prior to PSU change.
Parts:
- added C3, C4: 100nF, Capacitor_SMD:C_0402_1005Metric, symbol Device:C_Small
Connections:
- net +3.3V: now also C3.1, C4.1
- net GND: now also C3.2, C4.2
