File: BirdBox3/BirdBox3.kicad_sch (KiCad schematic)
At the start: 17 parts, among them J1 Raspberry Pi 2x20 Conn, J2 1x2 female, J2b 1x2 male, J4 1x6 female, J4 1x6 male, M1 Pimoroni Pico Lipo 4MB, M2 Wide-input Shim, SW1 Push button

Commit message: Deleted Run (reset) pushbutton:
- physical button was removed from the hatlet when Pico Lipo replaced Pico
- Pico Lipo has it's own on-board reset button
Parts:
- removed SW1: Push button, symbol Switch:SW_Push
Changed lines of the file:
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@@
-    (stroke (width 0) (type default) (color 0 0 0 0))
-  )
-  (wire (pts (xy 148.59 142.24) (xy 148.59 154.94))
     (stroke (width 0) (type default) (color 0 0 0 0))
   )
@@
   )
   (wire (pts (xy 121.92 55.88) (xy 138.43 55.88))
-    (stroke (width 0) (type default) (color 0 0 0 0))
-  )
-  (wire (pts (xy 119.38 142.24) (xy 148.59 142.24))
     (stroke (width 0) (type default) (color 0 0 0 0))
   )
@@
     (pin "9")
   )
-  (symbol (lib_id "power:GND") (at 148.59 165.1 0) (unit 1)
-    (in_bom yes) (on_board yes) (fields_autoplaced)
-    (property "Reference" "#PWR?" (id 0) (at 148.59 171.45 0)
-      (effects (font (size 1.27 1.27)) hide)
-    )
-    (property "Value" "GND" (id 1) (at 148.59 170.18 0))
-    (property "Footprint" "" (id 2) (at 148.59 165.1 0)
-      (effects (font (size 1.27 1.27)) hide)
-    )
-    (property "Datasheet" "" (id 3) (at 148.59 165.1 0)
-      (effects (font (size 1.27 1.27)) hide)
-    )
-    (pin "1")
-  )
   (symbol (lib_id "Connector:Conn_01x06_Male") (at 82.55 55.88 0) (unit 1)
     (in_bom yes) (on_board yes) (fields_autoplaced)
@@
     (pin "2")
   )
-  (symbol (lib_id "Switch:SW_Push") (at 148.59 160.02 270) (unit 1)
-    (in_bom yes) (on_board yes) (fields_autoplaced)
-    (property "Reference" "SW1" (id 0) (at 152.4 158.7499 90)
-      (effects (font (size 1.27 1.27)) (justify left))
-    )
-    (property "Value" "Push button" (id 1) (at 152.4 161.2899 90)
-      (effects (font (size 1.27 1.27)) (justify left))
-    )
-    (property "Footprint" "" (id 2) (at 153.67 160.02 0)
-      (effects (font (size 1.27 1.27)) hide)
-    )
-    (property "Datasheet" "~" (id 3) (at 153.67 160.02 0)
-      (effects (font (size 1.27 1.27)) hide)
-    )
-    (pin "1")
-    (pin "2")
-  )
   (symbol (lib_id "Device:R_Small") (at 209.55 66.04 0) (unit 1)
     (in_bom yes) (on_board yes)
@@
       (reference "#PWR0111") (unit 1) (value "+12V") (footprint "")
     )
-    (path "/14955393-9b87-4e5f-8c9d-3a54d04b273a"
-      (reference "#PWR?") (unit 1) (value "GND") (footprint "")
-    )
     (path "/6db16076-50f1-44dc-b1cd-dab3ad818a9d"
       (reference "#PWR?") (unit 1) (value "GND") (footprint "")
@@
       (reference "R5") (unit 1) (value "22 KOhm 1%") (footprint "")
     )
-    (path "/abf42133-0005-437b-9700-48463352169e"
-      (reference "SW1") (unit 1) (value "Push button") (footprint "")
-    )
-  )
+  )
